File: sampling-mesh-monitor.kicad_pcb (KiCad board)
At the start: 6 copper layers, 100 x 100 mm, 251 parts, among them J1 SWD, J2 SFP+, J3 USB_C_Receptacle_USB2.0, U1 OPA1656, U10 SKYA21003, U11 OPA1656, U12 TPS7B4253QPWPRQ1, U13 74LVC2G157, U14 AMS1117-3.3, U15 AMS1117-3.3, U16 AMS1117-3.3, U17 USBLC6-4SC6, U2 OPA1656, U3 TMUXHS4212, U4 TMUXHS4212, U5 LP2998, U6 PTN36241B, U7 STM32G474RBTx, U8 74LVC2G157, U9 SKYA21003, Y1 8MHz/20p

Commit message: PCB almost finished
Parts:
- removed logo_tu_darmstadt_25.0mm: G*****, logo_tu_darmstadt:logo_tu_darmstadt_25.0mm
- added GR1: TU Darmstadt logo, logo_tu_darmstadt:logo_tu_darmstadt_25.0mm, F.Cu at (149.8, 95.1)
- added Q1: AO3400A, Package_TO_SOT_SMD:SOT-23, F.Cu at (105.6, 103.9)
- added R100: 1k, Resistor_SMD:R_0402_1005Metric, F.Cu at (103.2, 128.7)
- added R101: 47k, Resistor_SMD:R_0402_1005Metric, F.Cu at (103.2, 126.3)
- added R99: 47, Resistor_SMD:R_0603_1608Metric, F.Cu at (101.7, 92.0)
- added TP13: VRB_DAC, TestPoint:TestPoint_Pad_1.5x1.5mm, F.Cu at (147.0, 77.1)
- added TP14: V_ADC2, TestPoint:TestPoint_Pad_1.5x1.5mm, F.Cu at (142.6, 99.2)
- added TP15: V_ADC1, TestPoint:TestPoint_Pad_1.5x1.5mm, F.Cu at (139.4, 100.0)
- added TP16: VRES_P, TestPoint:TestPoint_Pad_1.5x1.5mm, F.Cu at (105.6, 128.8)
- added TP17: VRES_N, TestPoint:TestPoint_Pad_1.5x1.5mm, F.Cu at (106.3, 93.7)
- added TP18: VBUS_SENSE, TestPoint:TestPoint_Pad_1.5x1.5mm, F.Cu at (185.7, 92.3)
- added TP19: VTIA, TestPoint:TestPoint_Pad_1.5x1.5mm, F.Cu at (119.7, 97.5)
- added TP20: PB2, TestPoint:TestPoint_Pad_1.5x1.5mm, F.Cu at (149.5, 76.3)
- added TP21: PB8, TestPoint:TestPoint_Pad_1.5x1.5mm, F.Cu at (177.8, 72.6)
- R11: value R -> 100
- R53: value 1k -> 22k
- R54: value 10k -> 47k
- R55: value R -> 22k
- R56, R8: value R -> 47k
- R7: value R -> 47; footprint Resistor_SMD:R_0402_1005Metric -> Resistor_SMD:R_0603_1608Metric
- R9: value R -> 10k
- TP1: value PA8 -> V_LVC_DAC
- TP2: value PA9 -> VB_DAC
- TP9: value PB6 -> PB4
- U5: footprint Package_SO:SO-8_3.9x4.9mm_P1.27mm -> footprints:SOIC-8-1EP_3.9x4.9mm_P1.27mm_EP2.34x2.34mm
- moved TP2 46.8 mm to (138.3, 128.2)
- moved TP1 35.8 mm to (175.5, 58.8)
- moved TP5 5.84 mm to (177.8, 75.1)
- moved TP9 5.81 mm to (173.5, 79.0)
- moved C53 5.65 mm to (130.1, 99.7), turned to 90 degrees
- moved R9 4.97 mm to (102.5, 97.5), turned to -90 degrees
- moved C52 3.08 mm to (132.5, 99.0), turned to 90 degrees
- moved D12 0.60 mm to (145.9, 107.8)
- moved R85 0.60 mm to (141.9, 107.8)
Connections:
- FB1 pad 1: VDDA -> Net-(U2B-+)
- J2 pad 7: /SFP5 -> /SFP6
- J2 pad 8: /SFP6 -> /SFP5
- R7 pad 2: GND -> Net-(Q1-D)
- R8 pad 1: /VRES -> /VRES_N
- TP1 pad 1: Net-(U7-PA8) -> /V_LVC_DAC
- TP2 pad 1: Net-(U7-PA9) -> /VBIAS_DAC
- TP9 pad 1: Net-(U7-PB6) -> Net-(U7-PB4)
- U1 pad 1: /VRES -> /VRES_N
- U10 pad 13: (no net) -> GND
- U12 pad 21: (no net) -> GND
- U2 pad 5: (no net) -> Net-(U2B-+)
- U2 pad 6: (no net) -> Net-(U2B--)
- U2 pad 7: (no net) -> /VRES_P
- U3 pad 21: (no net) -> GND
- U4 pad 21: (no net) -> GND
- U5 pad 2: (no net) -> unconnected-(U5-~{SD}-Pad2)
- U6 pad 13: (no net) -> +3.3VP
- U6 pad 25: (no net) -> GND
- U7 pad 26: /MESH_POL -> Net-(U7-PB2)
- U7 pad 33: /SFP5 -> /VTIA
- U7 pad 39: unconnected-(U7-PC7-Pad39) -> /VRES_EN
- U7 pad 42: Net-(U7-PA8) -> /VRES_N
- U7 pad 43: Net-(U7-PA9) -> /VRES_P
- U7 pad 55: unconnected-(U7-PD2-Pad55) -> /SFP5
- U7 pad 57: unconnected-(U7-PB4-Pad57) -> Net-(U7-PB4)
- U7 pad 59: Net-(U7-PB6) -> /SFP2
- U7 pad 61: /SFP2 -> Net-(U7-PB8)
- U9 pad 13: (no net) -> GND
Routing:
- net /VRES_P: track 0.00 -> 98.1 mm
- net /VRES_N: track 0.00 -> 93.2 mm, vias 0 -> 2
- net Net-(U2B-+): track 0.00 -> 72.6 mm
- net /VRES_EN: track 0.00 -> 67.8 mm
- net /VTIA: track 4.99 -> 64.3 mm
- net VBIAS: track 71.5 -> 96.4 mm
- net VRES_BIAS: track 33.2 -> 54.6 mm, vias 0 -> 2
- net GND: track 22.8 -> 39.5 mm, vias 450 -> 512
- net Net-(U7-PB2): track 0.00 -> 14.2 mm
- net Net-(U7-PB8): track 0.00 -> 13.4 mm
- net VDDA: track 154.5 -> 141.4 mm, vias 12 -> 11
- net Net-(U7-PB6): track 12.0 -> 0.00 mm
- net +3.3VP: track 49.8 -> 60.8 mm, vias 28 -> 29
- net Net-(U7-PA8): track 9.96 -> 0.00 mm
- net Net-(U7-PA9): track 7.25 -> 0.00 mm
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Other:
- outline, holes or cut-outs redrawn
- board text added: "Order parameters: JLCPCB 6 layer process, 1.2 mm total board thickness Stackup: JLC 06121H-3313 layer stackup, impedance controlled Surface finish: ENIG"

Commit message: Reannotate reference designators by PCB location
Parts:
- renumbered C56 to C1, C29 to C10, C39 to C11, C44 to C12, C40 to C13, C41 to C14, C42 to C15, C43 to C16, C36 to C17, C35 to C18, C45 to C19, C55 to C2, C46 to C20, C47 to C21, C48 to C22, C38 to C23, C26 to C24, C23 to C25, C27 to C26, C25 to C27, C24 to C28, C79 to C29, C57 to C3, C80 to C30, C3 to C31, C87 to C32, C37 to C33, C91 to C34, C88 to C35, C90 to C36, C81 to C37, C82 to C38, C32 to C39, C54 to C4, C31 to C40, C4 to C41, C5 to C42, C6 to C43, C18 to C44, C21 to C45, C20 to C46, C17 to C47, C22 to C48, C19 to C49, C59 to C5, C1 to C50, C30 to C52, C12 to C53, C83 to C54, C85 to C55, C86 to C56, C16 to C57, C84 to C58, C78 to C59, C58 to C6, C15 to C60, C2 to C61, C52 to C62, C53 to C63, C76 to C64, C77 to C65, C62 to C66, C63 to C67, C70 to C68, C71 to C69, C50 to C7, C9 to C70, C74 to C71, C60 to C72, C68 to C73, C11 to C74, C8 to C75, C34 to C76, C10 to C77, C75 to C78, C61 to C79, C49 to C8, C69 to C80, C14 to C81, C13 to C82, C33 to C83, C65 to C84, C64 to C85, C72 to C86, C73 to C87, C66 to C88, C67 to C89, C28 to C9, C7 to C90, D15 to D1, D2 to D10, D4 to D11, D11 to D12, D14 to D13, D13 to D14, D17 to D15, D12 to D16, D16 to D17, D10 to D2, D6 to D3, D9 to D4, D8 to D6, D1 to D8, D3 to D9, FB3 to FB2, FB4 to FB3, FB2 to FB4, H7 to H1, H1 to H2, H8 to H3, H3 to H5, H2 to H7, H5 to H8, J2 to J1, J3 to J2, J1 to J3, R19 to R1, R60 to R10, R31 to R100, R32 to R101, R77 to R11, R76 to R12, R35 to R13, R36 to R14, R26 to R15, R72 to R16, R73 to R17, R46 to R18, R71 to R19, R23 to R2, R74 to R20, R25 to R21, R13 to R22, R83 to R23, R81 to R24, R80 to R25, R82 to R26, R57 to R27, R45 to R28, R70 to R29, R15 to R3, R38 to R30, R37 to R31, R78 to R32, R17 to R33, R22 to R34, R12 to R35, R21 to R36, R18 to R37, R14 to R38, R58 to R39, R92 to R4, R61 to R40, R97 to R41, R66 to R42, R79 to R43, R98 to R44, R65 to R45, R88 to R46, R64 to R47, R62 to R48, R63 to R49, R20 to R5, R5 to R50, R50 to R51, R67 to R52, R3 to R53, R68 to R54, R52 to R55, R1 to R56, R2 to R57, R4 to R58, R47 to R59, R24 to R6, R69 to R60, R48 to R61, R51 to R62, R89 to R63, R99 to R64, R27 to R65, R28 to R66, R84 to R67, R87 to R68, R86 to R69, R16 to R7, R9 to R70, R8 to R71, R56 to R72, R55 to R73, R6 to R74, R53 to R75, R49 to R76, R54 to R77, R7 to R78, R10 to R79, R75 to R8, R91 to R80, R90 to R81, R94 to R82, R85 to R83, R11 to R84, R93 to R85, R101 to R86, R100 to R87, R42 to R88, R39 to R89, R59 to R9, R40 to R90, R43 to R91, R44 to R92, R33 to R93, R30 to R94, R29 to R97, R41 to R98, R34 to R99, TP12 to TP10, TP9 to TP11, TP11 to TP12, TP10 to TP13, TP3 to TP14, TP18 to TP15, TP17 to TP16, TP19 to TP17, TP15 to TP18, TP14 to TP19, TP7 to TP2, TP16 to TP20, TP2 to TP21, TP8 to TP3, TP13 to TP5, TP20 to TP7, TP5 to TP8, TP21 to TP9, U12 to U1, U17 to U10, U1 to U12, U2 to U13, U5 to U14, U16 to U15, U14 to U16, U15 to U17, U8 to U2, U13 to U3, U6 to U4, U9 to U5, U10 to U6, U3 to U7, U4 to U8, U7 to U9
