File: sampling-mesh-monitor.kicad_sch (KiCad schematic)
At the start: 262 parts, among them J1 SWD, J2 SFP+, J3 USB_C_Receptacle_USB2.0, T1 200ps, T10 200ps, T11 200ps, T12 200ps, T2 200ps, T3 200ps, T4 200ps, T5 200ps, T6 200ps, T7 200ps, T8 200ps, T9 200ps, U1 OPA1656, U10 SKYA21003, U11 OPA1656, U12 TPS7B4253QPWPRQ1, U13 74LVC2G157, U14 AMS1117-3.3, U15 AMS1117-3.3, U16 AMS1117-3.3, U17 USBLC6-4SC6, U2 OPA1656, U3 TMUXHS4212, U4 TMUXHS4212, U5 LP2998, U6 PTN36241B, U7 STM32G474RBTx, U8 74LVC2G157, U9 SKYA21003, Y1 8MHz/20p

Commit message: PCB almost finished
Parts:
- added GR1: TU Darmstadt logo, logo_tu_darmstadt:logo_tu_darmstadt_25.0mm, symbol Graphic:SYM_Flash_Small
- added Q1: AO3400A, Package_TO_SOT_SMD:SOT-23, symbol Transistor_FET:AO3400A
- added R100: 1k, Resistor_SMD:R_0402_1005Metric, symbol Device:R
- added R101: 47k, Resistor_SMD:R_0402_1005Metric, symbol Device:R
- added R99: 47, Resistor_SMD:R_0603_1608Metric, symbol Device:R
- added TP13: VRB_DAC, TestPoint:TestPoint_Pad_1.5x1.5mm, symbol Connector:TestPoint
- added TP14: V_ADC2, TestPoint:TestPoint_Pad_1.5x1.5mm, symbol Connector:TestPoint
- added TP15: V_ADC1, TestPoint:TestPoint_Pad_1.5x1.5mm, symbol Connector:TestPoint
- added TP16: VRES_P, TestPoint:TestPoint_Pad_1.5x1.5mm, symbol Connector:TestPoint
- added TP17: VRES_N, TestPoint:TestPoint_Pad_1.5x1.5mm, symbol Connector:TestPoint
- added TP18: VBUS_SENSE, TestPoint:TestPoint_Pad_1.5x1.5mm, symbol Connector:TestPoint
- added TP19: VTIA, TestPoint:TestPoint_Pad_1.5x1.5mm, symbol Connector:TestPoint
- added TP20: PB2, TestPoint:TestPoint_Pad_1.5x1.5mm, symbol Connector:TestPoint
- added TP21: PB8, TestPoint:TestPoint_Pad_1.5x1.5mm, symbol Connector:TestPoint
- added unit 2 of U2
- R11: value R -> 100; LCSC (none) -> C25076
- R30, R33, R40, R43: now left out of the parts list
- R53: value 1k -> 22k; LCSC C11702 -> C25768
- R54: value 10k -> 47k; LCSC C2654005 -> C25792
- R55: value R -> 22k; LCSC (none) -> C25768
- R56, R8: value R -> 47k; LCSC (none) -> C25792
- R7: value R -> 47; footprint Resistor_SMD:R_0402_1005Metric -> Resistor_SMD:R_0603_1608Metric; LCSC (none) -> C23182
- R9: value R -> 10k; LCSC (none) -> C2654005
- TP1: value PA8 -> V_LVC_DAC
- TP2: value PA9 -> VB_DAC
- TP9: value PB6 -> PB4
- U5: footprint Package_SO:SO-8_3.9x4.9mm_P1.27mm -> footprints:SOIC-8-1EP_3.9x4.9mm_P1.27mm_EP2.34x2.34mm
Connections:
- net VRES is gone; now on net VRES_N: R8.1, U1.1
- net +3.3VP: now also U6.13 (VDD)
- net GND: now also U10.13 (GND), U12.21 (GND), U3.21 (GND), U4.21 (GND), U5.9 (GND), U6.25 (GND), U9.13 (GND), Q1.2 (S); no longer R7.2, U10.EP (GND), U12.EP (GND), U3.EP (GND), U4.EP (GND), U5.EP (GND), U6.EP (GND), U9.EP (GND)
- net SFP2: now also U7.59 (PB6); no longer U7.61 (PB8)
- net SFP5: now also J2.8 (Pin_8), U7.55 (PD2); no longer J2.7 (Pin_7), U7.33 (PB11)
- net SFP6: now also J2.7 (Pin_7); no longer J2.8 (Pin_8)
- net VBIAS_DAC: now also TP2.1
- net VBUS_SENSE: now also TP18.1
- net VDDA: now also R99.1; no longer FB1.1
- net VRES_BIAS: now also R100.2
- net VRES_BIAS_DAC: now also TP13.1
- net VTIA: now also U7.33 (PB11), TP19.1
- net V_ADC1: now also TP15.1
- net V_ADC2: now also TP14.1
- net V_LVC_DAC: now also TP1.1
- net VRES_N: now reaches U7.42 (PA8)
- net VRES_N: now also TP17.1; no longer TP1.1
- net VRES_P: now reaches U7.43 (PA9)
- net VRES_P: now also R101.1, TP16.1, U2.7; no longer TP2.1
- net VRES_EN: now reaches U7.39 (PC7)
- net VRES_EN: now also Q1.1 (G)
- net at U7.57 (PB4): now also TP9.1
- net MESH_POL: no longer names the net of U7.26 (PB2)
- net MESH_POL: now also TP20.1
- new net: Q1.3 (D), R7.2
- new net: FB1.1, R99.2, U2.5 (+)
- new net: R100.1, R101.2, U2.6 (-)
- new net: TP21.1, U7.61 (PB8)
Other:
- moved on the sheet: C2, R10, U1B

Commit message: Reannotate reference designators by PCB location
Parts:
- renumbered C56 to C1, C29 to C10, C39 to C11, C44 to C12, C40 to C13, C41 to C14, C42 to C15, C43 to C16, C36 to C17, C35 to C18, C45 to C19, C55 to C2, C46 to C20, C47 to C21, C48 to C22, C38 to C23, C26 to C24, C23 to C25, C27 to C26, C25 to C27, C24 to C28, C79 to C29, C57 to C3, C80 to C30, C3 to C31, C87 to C32, C37 to C33, C91 to C34, C88 to C35, C90 to C36, C81 to C37, C82 to C38, C32 to C39, C54 to C4, C31 to C40, C4 to C41, C5 to C42, C6 to C43, C18 to C44, C21 to C45, C20 to C46, C17 to C47, C22 to C48, C19 to C49, C59 to C5, C1 to C50, C30 to C52, C12 to C53, C83 to C54, C85 to C55, C86 to C56, C16 to C57, C84 to C58, C78 to C59, C58 to C6, C15 to C60, C2 to C61, C52 to C62, C53 to C63, C76 to C64, C77 to C65, C62 to C66, C63 to C67, C70 to C68, C71 to C69, C50 to C7, C9 to C70, C74 to C71, C60 to C72, C68 to C73, C11 to C74, C8 to C75, C34 to C76, C10 to C77, C75 to C78, C61 to C79, C49 to C8, C69 to C80, C14 to C81, C13 to C82, C33 to C83, C65 to C84, C64 to C85, C72 to C86, C73 to C87, C66 to C88, C67 to C89, C28 to C9, C7 to C90, D15 to D1, D2 to D10, D4 to D11, D11 to D12, D14 to D13, D13 to D14, D17 to D15, D12 to D16, D16 to D17, D10 to D2, D6 to D3, D9 to D4, D8 to D6, D1 to D8, D3 to D9, FB3 to FB2, FB4 to FB3, FB2 to FB4, H7 to H1, H1 to H2, H8 to H3, H3 to H5, H2 to H7, H5 to H8, J2 to J1, J3 to J2, J1 to J3, R19 to R1, R60 to R10, R31 to R100, R32 to R101, R77 to R11, R76 to R12, R35 to R13, R36 to R14, R26 to R15, R72 to R16, R73 to R17, R46 to R18, R71 to R19, R23 to R2, R74 to R20, R25 to R21, R13 to R22, R83 to R23, R81 to R24, R80 to R25, R82 to R26, R57 to R27, R45 to R28, R70 to R29, R15 to R3, R38 to R30, R37 to R31, R78 to R32, R17 to R33, R22 to R34, R12 to R35, R21 to R36, R18 to R37, R14 to R38, R58 to R39, R92 to R4, R61 to R40, R97 to R41, R66 to R42, R79 to R43, R98 to R44, R65 to R45, R88 to R46, R64 to R47, R62 to R48, R63 to R49, R20 to R5, R5 to R50, R50 to R51, R67 to R52, R3 to R53, R68 to R54, R52 to R55, R1 to R56, R2 to R57, R4 to R58, R47 to R59, R24 to R6, R69 to R60, R48 to R61, R51 to R62, R89 to R63, R99 to R64, R27 to R65, R28 to R66, R84 to R67, R87 to R68, R86 to R69, R16 to R7, R9 to R70, R8 to R71, R56 to R72, R55 to R73, R6 to R74, R53 to R75, R49 to R76, R54 to R77, R7 to R78, R10 to R79, R75 to R8, R91 to R80, R90 to R81, R94 to R82, R85 to R83, R11 to R84, R93 to R85, R101 to R86, R100 to R87, R42 to R88, R39 to R89, R59 to R9, R40 to R90, R43 to R91, R44 to R92, R33 to R93, R30 to R94, R29 to R97, R41 to R98, R34 to R99, TP12 to TP10, TP9 to TP11, TP11 to TP12, TP10 to TP13, TP3 to TP14, TP18 to TP15, TP17 to TP16, TP19 to TP17, TP15 to TP18, TP14 to TP19, TP7 to TP2, TP16 to TP20, TP2 to TP21, TP8 to TP3, TP13 to TP5, TP20 to TP7, TP5 to TP8, TP21 to TP9, U12 to U1, U17 to U10, U1 to U12, U2 to U13, U5 to U14, U16 to U15, U14 to U16, U15 to U17, U8 to U2, U13 to U3, U6 to U4, U9 to U5, U10 to U6, U3 to U7, U4 to U8, U7 to U9
