File: uut_mesh_board_cal/uut_mesh_board_cal.kicad_pcb (KiCad board)
At the start: 2 copper layers, 36.5 x 36.5 mm, 11 parts, among them J1 Conn_02x10_Counter_Clockwise, J2 Conn_02x10_Counter_Clockwise, J3 Conn_02x10_Counter_Clockwise, J4 Conn_02x10_Counter_Clockwise

Commit message: uut/cal kit: Add version number
Other:
- board text added: "Sampling Mesh Monitor Cal kit v1"
- board text removed: "Sampling Mesh Monitor Cal kit"
