File: uut_meshes/uut_meshes.kicad_pcb (KiCad board)
At the start: 4 copper layers, 100 x 100 mm, 5 parts, among them J1 Conn_02x10_Counter_Clockwise, J2 Conn_02x10_Counter_Clockwise, J3 Conn_02x10_Counter_Clockwise, J4 Conn_02x10_Counter_Clockwise

Commit message: Mesh test board WIP
Parts:
- removed logo_tu_darmstadt_30.0mm: G*****, logo_tu_darmstadt:logo_tu_darmstadt_30.0mm
- added J10: Conn_02x04_Top_Bottom, PCM_kimesh_anchors_2wire:MeshAnchor_2W_T0.120mm_S0.120mm, B.Cu at (185.0, 124.5)
- added J11: Conn_02x04_Top_Bottom, PCM_kimesh_anchors_2wire:MeshAnchor_2W_T0.120mm_S0.120mm, B.Cu at (185.0, 114.5)
- added J12: Conn_02x04_Top_Bottom, PCM_kimesh_anchors_2wire:MeshAnchor_2W_T0.120mm_S0.120mm, B.Cu at (185.0, 96.5)
- added J5: Conn_02x04_Top_Bottom, PCM_kimesh_anchors_2wire:MeshAnchor_2W_T0.120mm_S0.120mm, F.Cu at (115.5, 65.0)
- added J6: Conn_02x04_Top_Bottom, PCM_kimesh_anchors_2wire:MeshAnchor_2W_T0.120mm_S0.120mm, F.Cu at (184.5, 65.0)
- added J7: Conn_02x04_Top_Bottom, PCM_kimesh_anchors_2wire:MeshAnchor_2W_T0.120mm_S0.120mm, B.Cu at (185.0, 134.5)
- added J9: Conn_02x04_Top_Bottom, PCM_kimesh_anchors_2wire:MeshAnchor_2W_T0.120mm_S0.120mm, B.Cu at (185.0, 130.5)
- added R1: 0, Resistor_SMD:R_0402_1005Metric, F.Cu at (186.9, 135.0)
- added R10: 0, Resistor_SMD:R_0402_1005Metric, F.Cu at (188.1, 130.6)
- added R11: 0, Resistor_SMD:R_0402_1005Metric, F.Cu at (185.7, 127.9)
- added R12: 0, Resistor_SMD:R_0402_1005Metric, F.Cu at (186.9, 127.9)
- added R13: 0, Resistor_SMD:R_0402_1005Metric, F.Cu at (188.1, 127.9)
- added R14: 0, Resistor_SMD:R_0402_1005Metric, F.Cu at (189.3, 127.9)
- added R15: 0, Resistor_SMD:R_0402_1005Metric, F.Cu at (189.3, 123.5)
- added R16: 0, Resistor_SMD:R_0402_1005Metric, F.Cu at (188.1, 123.5)
- added R17: 0, Resistor_SMD:R_0402_1005Metric, F.Cu at (186.9, 125.7)
- added R18: 0, Resistor_SMD:R_0402_1005Metric, F.Cu at (185.7, 125.7)
- added R19: 0, Resistor_SMD:R_0402_1005Metric, F.Cu at (188.1, 125.7)
- added R2: 0, Resistor_SMD:R_0402_1005Metric, F.Cu at (185.7, 135.0)
- added R20: 0, Resistor_SMD:R_0402_1005Metric, F.Cu at (189.3, 125.7)
- added R21: 0, Resistor_SMD:R_0402_1005Metric, F.Cu at (185.7, 120.2)
- added R22: 0, Resistor_SMD:R_0402_1005Metric, F.Cu at (186.9, 120.2)
- added R23: 0, Resistor_SMD:R_0402_1005Metric, F.Cu at (188.1, 120.2)
- added R24: 0, Resistor_SMD:R_0402_1005Metric, F.Cu at (189.3, 120.2)
- added R25: 0, Resistor_SMD:R_0402_1005Metric, F.Cu at (189.3, 115.8)
- added R26: 0, Resistor_SMD:R_0402_1005Metric, F.Cu at (188.1, 115.8)
- added R27: 0, Resistor_SMD:R_0402_1005Metric, F.Cu at (186.9, 118.0)
- added R28: 0, Resistor_SMD:R_0402_1005Metric, F.Cu at (185.7, 118.0)
- added R29: 0, Resistor_SMD:R_0402_1005Metric, F.Cu at (188.1, 118.0)
- added R3: 0, Resistor_SMD:R_0402_1005Metric, F.Cu at (188.1, 135.0)
- added R30: 0, Resistor_SMD:R_0402_1005Metric, F.Cu at (189.3, 118.0)
- added R31: 0, Resistor_SMD:R_0402_1005Metric, F.Cu at (185.7, 112.3)
- added R32: 0, Resistor_SMD:R_0402_1005Metric, F.Cu at (186.9, 112.3)
- added R33: 0, Resistor_SMD:R_0402_1005Metric, F.Cu at (188.1, 112.3)
- added R34: 0, Resistor_SMD:R_0402_1005Metric, F.Cu at (189.3, 112.3)
- added R35: 0, Resistor_SMD:R_0402_1005Metric, F.Cu at (189.3, 108.0)
- added R36: 0, Resistor_SMD:R_0402_1005Metric, F.Cu at (188.1, 108.0)
- added R37: 0, Resistor_SMD:R_0402_1005Metric, F.Cu at (186.9, 110.2)
- added R38: 0, Resistor_SMD:R_0402_1005Metric, F.Cu at (185.7, 110.2)
- added R39: 0, Resistor_SMD:R_0402_1005Metric, F.Cu at (188.1, 110.2)
- added R4: 0, Resistor_SMD:R_0402_1005Metric, F.Cu at (189.3, 135.0)
- added R40: 0, Resistor_SMD:R_0402_1005Metric, F.Cu at (189.3, 110.2)
- added R5: 0, Resistor_SMD:R_0402_1005Metric, F.Cu at (185.7, 132.8)
- added R6: 0, Resistor_SMD:R_0402_1005Metric, F.Cu at (186.9, 132.8)
- added R7: 0, Resistor_SMD:R_0402_1005Metric, F.Cu at (189.3, 132.8)
- added R8: 0, Resistor_SMD:R_0402_1005Metric, F.Cu at (188.1, 132.8)
- added R9: 0, Resistor_SMD:R_0402_1005Metric, F.Cu at (189.3, 130.6)
Connections:
- J1 pad 17: Net-(J1-Pin_15) -> Net-(J1-Pin_17)
- J1 pad 19: Net-(J1-Pin_13) -> Net-(J1-Pin_19)
- J3 pad 13: Net-(J3-Pin_13) -> unconnected-(J3-Pin_13-Pad13)
- J3 pad 15: Net-(J3-Pin_15) -> unconnected-(J3-Pin_15-Pad15)
- J3 pad 17: Net-(J3-Pin_17) -> unconnected-(J3-Pin_17-Pad17)
- J3 pad 19: Net-(J3-Pin_19) -> unconnected-(J3-Pin_19-Pad19)
- J4 pad 13: unconnected-(J4-Pin_13-Pad13) -> Net-(J4-Pin_13)
- J4 pad 15: unconnected-(J4-Pin_15-Pad15) -> Net-(J4-Pin_15)
- J4 pad 17: unconnected-(J4-Pin_17-Pad17) -> Net-(J4-Pin_17)
- J4 pad 19: unconnected-(J4-Pin_19-Pad19) -> Net-(J4-Pin_19)
Routing:
- net GND: track 446.2 -> 406.3 mm, vias 56 -> 57
- net Net-(J2-Pin_17): track 0.00 -> 19.4 mm
- net Net-(J2-Pin_19): track 0.00 -> 16.8 mm
- net Net-(J2-Pin_13): track 0.00 -> 16.4 mm
- net Net-(J4-Pin_17): track 0.00 -> 15.8 mm
- net Net-(J1-Pin_19): track 0.00 -> 15.7 mm
- net Net-(J4-Pin_19): track 0.00 -> 15.6 mm
- net Net-(J2-Pin_15): track 0.00 -> 15.4 mm
- net Net-(J4-Pin_15): track 0.00 -> 15.4 mm
- net Net-(J1-Pin_17): track 0.00 -> 15.3 mm
- net Net-(J4-Pin_13): track 0.00 -> 15.2 mm
- net Net-(J1-Pin_15): track 0.00 -> 15.1 mm
- net Net-(J1-Pin_13): track 0.00 -> 15.0 mm
- net Net-(R28-Pad1): track 0.00 -> 11.3 mm
- net Net-(R18-Pad1): track 0.00 -> 11.2 mm
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
Commit message: meshes WIP
Parts:
- added J10: Conn_02x04_Top_Bottom, PCM_kimesh_anchors_2wire:MeshAnchor_2W_T0.120mm_S0.120mm, B.Cu at (115.0, 124.5)
- added J11: Conn_02x04_Top_Bottom, PCM_kimesh_anchors_2wire:MeshAnchor_2W_T0.120mm_S0.120mm, B.Cu at (115.0, 114.5)
- added J12: Conn_02x04_Top_Bottom, PCM_kimesh_anchors_2wire:MeshAnchor_2W_T0.120mm_S0.120mm, B.Cu at (115.0, 96.5)
- added J7: Conn_02x04_Top_Bottom, PCM_kimesh_anchors_2wire:MeshAnchor_2W_T0.120mm_S0.120mm, B.Cu at (115.0, 133.5)
- added J9: Conn_02x04_Top_Bottom, PCM_kimesh_anchors_2wire:MeshAnchor_2W_T0.120mm_S0.120mm, B.Cu at (115.0, 127.5)
- added R1: 0, Resistor_SMD:R_0402_1005Metric, F.Cu at (111.4, 134.6)
- added R10: 0, Resistor_SMD:R_0402_1005Metric, F.Cu at (112.6, 130.2)
- added R11: 0, Resistor_SMD:R_0402_1005Metric, F.Cu at (110.2, 127.5)
- added R12: 0, Resistor_SMD:R_0402_1005Metric, F.Cu at (111.4, 127.5)
- added R13: 0, Resistor_SMD:R_0402_1005Metric, F.Cu at (112.6, 127.5)
- added R14: 0, Resistor_SMD:R_0402_1005Metric, F.Cu at (113.8, 127.5)
- added R15: 0, Resistor_SMD:R_0402_1005Metric, F.Cu at (113.8, 123.1)
- added R16: 0, Resistor_SMD:R_0402_1005Metric, F.Cu at (112.6, 123.1)
- added R17: 0, Resistor_SMD:R_0402_1005Metric, F.Cu at (111.4, 125.3)
- added R18: 0, Resistor_SMD:R_0402_1005Metric, F.Cu at (110.2, 125.3)
- added R19: 0, Resistor_SMD:R_0402_1005Metric, F.Cu at (112.6, 125.3)
- added R2: 0, Resistor_SMD:R_0402_1005Metric, F.Cu at (110.2, 134.6)
- added R20: 0, Resistor_SMD:R_0402_1005Metric, F.Cu at (113.8, 125.3)
- added R21: 0, Resistor_SMD:R_0402_1005Metric, F.Cu at (110.2, 119.8)
- added R22: 0, Resistor_SMD:R_0402_1005Metric, F.Cu at (111.4, 119.8)
- added R23: 0, Resistor_SMD:R_0402_1005Metric, F.Cu at (112.6, 119.8)
- added R24: 0, Resistor_SMD:R_0402_1005Metric, F.Cu at (113.8, 119.8)
- added R25: 0, Resistor_SMD:R_0402_1005Metric, F.Cu at (113.8, 115.4)
- added R26: 0, Resistor_SMD:R_0402_1005Metric, F.Cu at (112.6, 115.4)
- added R27: 0, Resistor_SMD:R_0402_1005Metric, F.Cu at (111.4, 117.6)
- added R28: 0, Resistor_SMD:R_0402_1005Metric, F.Cu at (110.2, 117.6)
- added R29: 0, Resistor_SMD:R_0402_1005Metric, F.Cu at (112.6, 117.6)
- added R3: 0, Resistor_SMD:R_0402_1005Metric, F.Cu at (112.6, 134.6)
- added R30: 0, Resistor_SMD:R_0402_1005Metric, F.Cu at (113.8, 117.6)
- added R31: 0, Resistor_SMD:R_0402_1005Metric, F.Cu at (110.2, 112.0)
- added R32: 0, Resistor_SMD:R_0402_1005Metric, F.Cu at (111.4, 112.0)
- added R33: 0, Resistor_SMD:R_0402_1005Metric, F.Cu at (112.6, 112.0)
- added R34: 0, Resistor_SMD:R_0402_1005Metric, F.Cu at (113.8, 112.0)
- added R35: 0, Resistor_SMD:R_0402_1005Metric, F.Cu at (113.8, 107.5)
- added R36: 0, Resistor_SMD:R_0402_1005Metric, F.Cu at (112.6, 107.5)
- added R37: 0, Resistor_SMD:R_0402_1005Metric, F.Cu at (111.4, 109.8)
- added R38: 0, Resistor_SMD:R_0402_1005Metric, F.Cu at (110.2, 109.8)
- added R39: 0, Resistor_SMD:R_0402_1005Metric, F.Cu at (112.6, 109.8)
- added R4: 0, Resistor_SMD:R_0402_1005Metric, F.Cu at (113.8, 134.6)
- added R40: 0, Resistor_SMD:R_0402_1005Metric, F.Cu at (113.8, 109.8)
- added R5: 0, Resistor_SMD:R_0402_1005Metric, F.Cu at (110.2, 132.4)
- added R6: 0, Resistor_SMD:R_0402_1005Metric, F.Cu at (111.4, 132.4)
- added R7: 0, Resistor_SMD:R_0402_1005Metric, F.Cu at (113.8, 132.4)
- added R8: 0, Resistor_SMD:R_0402_1005Metric, F.Cu at (112.6, 132.4)
- added R9: 0, Resistor_SMD:R_0402_1005Metric, F.Cu at (113.8, 130.2)
Connections:
- net Net-(J11-Pin_5) renamed /M3B
- net Net-(J11-Pin_6) renamed /M3A
- net Net-(J5-Pin_5) renamed /M6A
- net Net-(J5-Pin_6) renamed /M6B
- net Net-(J7-Pin_5) renamed /M0B
- net Net-(J7-Pin_6) renamed /M0A
- net Net-(J9-Pin_5) renamed /M1B
- net Net-(J9-Pin_6) renamed /M1A
- R10 pad 2: Net-(J2-Pin_17) -> Net-(R10-Pad2)
- R19 pad 1: Net-(R17-Pad1) -> Net-(R19-Pad1)
- R2 pad 1: Net-(J7-Pin_1) -> Net-(J7-Pin_4)
- R2 pad 2: Net-(J2-Pin_13) -> Net-(R2-Pad2)
- R20 pad 1: Net-(R18-Pad1) -> Net-(R20-Pad1)
- R21 pad 1: Net-(J10-Pin_1) -> Net-(R21-Pad1)
- R21 pad 2: Net-(R18-Pad1) -> Net-(R20-Pad1)
- R22 pad 1: Net-(J10-Pin_2) -> Net-(R22-Pad1)
- R22 pad 2: Net-(R17-Pad1) -> Net-(R19-Pad1)
- R23 pad 1: Net-(J10-Pin_3) -> Net-(R23-Pad1)
- R24 pad 1: Net-(J10-Pin_4) -> Net-(R24-Pad1)
- R27 pad 2: Net-(R17-Pad1) -> Net-(R19-Pad1)
- R29 pad 2: Net-(J10-Pin_3) -> Net-(R23-Pad1)
- R3 pad 1: Net-(J7-Pin_3) -> Net-(J7-Pin_2)
- R3 pad 2: Net-(J2-Pin_17) -> Net-(R10-Pad2)
- R38 pad 2: Net-(R28-Pad1) -> Net-(R38-Pad2)
- R4 pad 1: Net-(J7-Pin_4) -> Net-(J7-Pin_1)
- R4 pad 2: Net-(J2-Pin_19) -> Net-(R4-Pad2)
- R6 pad 2: Net-(J2-Pin_15) -> Net-(R6-Pad2)
- R7 pad 2: Net-(J7-Pin_4) -> Net-(J7-Pin_1)
- R8 pad 2: Net-(J7-Pin_3) -> Net-(J7-Pin_2)
Routing:
- net Net-(R38-Pad1): track 4.02 -> 37.5 mm, vias 0 -> 2
- net Net-(R37-Pad1): track 1.20 -> 27.9 mm, vias 0 -> 2
- net Net-(R36-Pad1): track 0.00 -> 25.0 mm, vias 0 -> 2
- net Net-(R35-Pad1): track 0.00 -> 21.2 mm, vias 0 -> 2
- net unconnected-(J3-Pin_19-Pad19): track 0.00 -> 14.9 mm
- net Net-(J2-Pin_13): track 16.4 -> 30.5 mm
- net unconnected-(J3-Pin_17-Pad17): track 0.00 -> 14.1 mm
- net unconnected-(J3-Pin_15-Pad15): track 0.00 -> 13.4 mm
- net Net-(J7-Pin_2): track 0.00 -> 11.9 mm, vias 0 -> 4
- net Net-(R28-Pad1): track 11.3 -> 22.7 mm
- net Net-(R18-Pad1): track 11.2 -> 22.4 mm
- net Net-(R11-Pad2): track 10.6 -> 21.2 mm
- net Net-(J7-Pin_4): track 1.54 -> 11.5 mm, vias 0 -> 2
- net Net-(R26-Pad1): track 9.58 -> 19.2 mm
- net Net-(R16-Pad1): track 9.49 -> 19.0 mm
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