File: uut_meshes/uut_meshes.kicad_sch (KiCad schematic)
At the start: 4 parts, among them J1 Conn_02x10_Counter_Clockwise, J2 Conn_02x10_Counter_Clockwise, J3 Conn_02x10_Counter_Clockwise, J4 Conn_02x10_Counter_Clockwise

Commit message: Mesh test board WIP
Parts:
- added J10, J11, J12, J5, J6, J7, J9: Conn_02x04_Top_Bottom, PCM_kimesh_anchors_2wire:MeshAnchor_2W_T0.120mm_S0.120mm, symbol Connector_Generic:Conn_02x04_Top_Bottom
- added R1, R10, R11, R12, R13, R14, R15, R16, R17, R18, R19, R2, R20, R21, R22, R23, R24, R25, R26, R27, R28, R29, R3, R30, R31, R32, R33, R34, R35, R36, R37, R38, R39, R4, R40, R5, R6, R7, R8, R9: 0, Resistor_SMD:R_0603_1608Metric, symbol Device:R
- J2: now left out of the parts list
Connections:
- net at J2.13 (Pin_13): now also R2.2, R5.2
- net at J2.15 (Pin_15): now also R1.2, R6.2
- net at J2.17 (Pin_17): now also R10.2, R3.2
- net at J2.19 (Pin_19): now also R4.2, R9.2
- net at J4.13 (Pin_13): now also J5.1 (Pin_1)
- net at J4.15 (Pin_15): now also J5.2 (Pin_2)
- net at J4.17 (Pin_17): now also J5.3 (Pin_3)
- net at J4.19 (Pin_19): now also J5.4 (Pin_4)
- net at J1.13 (Pin_13): now also J6.1 (Pin_1)
- net at J1.15 (Pin_15): now also J6.2 (Pin_2)
- net at J1.17 (Pin_17): now also J6.3 (Pin_3)
- net at J1.19 (Pin_19): now also J6.4 (Pin_4)
- new net: R17.1, R19.1, R22.2, R27.2
- new net: J9.3 (Pin_3), R13.1, R19.2
- new net: R12.2, R17.2, R6.1, R8.1
- new net: J7.2 (Pin_2), R3.1, R8.2
- new net: J10.4 (Pin_4), R24.1, R30.2
- new net: R15.1, R24.2, R25.2
- new net: J12.3 (Pin_3), R36.1
- new net: R26.1, R33.2, R36.2
- new net: J10.2 (Pin_2), R22.1
- new net: J9.1 (Pin_1), R11.1
- new net: R11.2, R18.2, R5.1, R7.1
- new net: R27.1, R29.1, R32.2, R37.2
- new net: R16.1, R23.2, R26.2
- new net: R10.1, R13.2, R16.2
- new net: J11.1 (Pin_1), R31.1
- new net: J11.2 (Pin_2), R32.1
- new net: J11.3 (Pin_3), R33.1, R39.2
- new net: J11.4 (Pin_4), R34.1, R40.2
- new net: J9.4 (Pin_4), R14.1, R20.2
- new net: R14.2, R15.2, R9.1
- new net: R28.1, R30.1, R31.2, R38.2
- new net: R18.1, R20.1, R21.2, R28.2
- new net: J10.1 (Pin_1), R21.1
- new net: J12.4 (Pin_4), R35.1
- new net: R25.1, R34.2, R35.2
- new net: J12.2 (Pin_2), R37.1, R39.1
- new net: J10.3 (Pin_3), R23.1, R29.2
- new net: J12.1 (Pin_1), R38.1, R40.1
- new net: J9.2 (Pin_2), R12.1
- new net: J7.1 (Pin_1), R4.1, R7.2
- new net: J7.3 (Pin_3), R1.1
- new net: J7.4 (Pin_4), R2.1
- new net M0A: J7.6 (Pin_6), J7.7 (Pin_7)
- new net M0B: J7.5 (Pin_5), J7.8 (Pin_8)
- new net M1A: J9.6 (Pin_6), J9.7 (Pin_7)
- new net M1B: J9.5 (Pin_5), J9.8 (Pin_8)
- new net M2A: J10.6 (Pin_6), J10.7 (Pin_7)
- new net M2B: J10.5 (Pin_5), J10.8 (Pin_8)
- new net M3A: J11.6 (Pin_6), J11.7 (Pin_7)
- new net M3B: J11.5 (Pin_5), J11.8 (Pin_8)
- new net M4A: J12.6 (Pin_6), J12.7 (Pin_7)
- new net M4B: J12.5 (Pin_5), J12.8 (Pin_8)
- new net M5A: J6.5 (Pin_5), J6.8 (Pin_8)
- new net M5B: J6.6 (Pin_6), J6.7 (Pin_7)
- new net M6A: J5.5 (Pin_5), J5.8 (Pin_8)
- new net M6B: J5.6 (Pin_6), J5.7 (Pin_7)
Other:
- moved on the sheet: J2, J3, J4

Commit message: meshes WIP
Parts:
- R10, R11, R12, R14, R15, R16, R19, R2, R20, R21, R22, R23, R24, R25, R26, R27, R29, R3, R33, R34, R35, R37, R38, R39, R4, R40, R6, R7, R8: footprint Resistor_SMD:R_0603_1608Metric -> Resistor_SMD:R_0402_1005Metric
Changed lines of the file:
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@@
 			)
 		)
-		(property "Footprint" "Resistor_SMD:R_0603_1608Metric"
+		(property "Footprint" "Resistor_SMD:R_0402_1005Metric"
 			(at 218.44 94.742 90)
 			(effects
@@
 			)
 		)
-		(property "Footprint" "Resistor_SMD:R_0603_1608Metric"
+		(property "Footprint" "Resistor_SMD:R_0402_1005Metric"
 			(at 176.53 94.742 90)
 			(effects
@@
 			)
 		)
-		(property "Footprint" "Resistor_SMD:R_0603_1608Metric"
+		(property "Footprint" "Resistor_SMD:R_0402_1005Metric"
 			(at 255.778 87.63 90)
 			(effects
@@
 			)
 		)
-		(property "Footprint" "Resistor_SMD:R_0603_1608Metric"
+		(property "Footprint" "Resistor_SMD:R_0402_1005Metric"
 			(at 245.618 87.63 90)
 			(effects
@@
 			)
 		)
-		(property "Footprint" "Resistor_SMD:R_0603_1608Metric"
+		(property "Footprint" "Resistor_SMD:R_0402_1005Metric"
 			(at 176.53 69.342 90)
 			(effects
@@
 			)
 		)
-		(property "Footprint" "Resistor_SMD:R_0603_1608Metric"
+		(property "Footprint" "Resistor_SMD:R_0402_1005Metric"
 			(at 198.628 87.63 90)
 			(effects
@@
 			)
 		)
-		(property "Footprint" "Resistor_SMD:R_0603_1608Metric"
+		(property "Footprint" "Resistor_SMD:R_0402_1005Metric"
 			(at 260.35 69.342 90)
 			(effects
@@
 			)
 		)
-		(property "Footprint" "Resistor_SMD:R_0603_1608Metric"
+		(property "Footprint" "Resistor_SMD:R_0402_1005Metric"
 			(at 260.35 64.262 90)
 			(effects
@@
 			)
 		)
-		(property "Footprint" "Resistor_SMD:R_0603_1608Metric"
+		(property "Footprint" "Resistor_SMD:R_0402_1005Metric"
 			(at 218.44 64.262 90)
 			(effects
@@
 			)
 		)
-		(property "Footprint" "Resistor_SMD:R_0603_1608Metric"
+		(property "Footprint" "Resistor_SMD:R_0402_1005Metric"
 			(at 213.868 87.63 90)
 			(effects
@@
 			)
 		)
-		(property "Footprint" "Resistor_SMD:R_0603_1608Metric"
+		(property "Footprint" "Resistor_SMD:R_0402_1005Metric"
 			(at 292.608 87.63 90)
 			(effects
@@
 			)
 		)
-		(property "Footprint" "Resistor_SMD:R_0603_1608Metric"
+		(property "Footprint" "Resistor_SMD:R_0402_1005Metric"
 			(at 176.53 64.262 90)
 			(effects
@@
 			)
 		)
-		(property "Footprint" "Resistor_SMD:R_0603_1608Metric"
+		(property "Footprint" "Resistor_SMD:R_0402_1005Metric"
 			(at 240.538 87.63 90)
 			(effects
@@
 			)
 		)
-		(property "Footprint" "Resistor_SMD:R_0603_1608Metric"
+		(property "Footprint" "Resistor_SMD:R_0402_1005Metric"
 			(at 302.26 59.182 90)
 			(effects
@@
 			)
 		)
-		(property "Footprint" "Resistor_SMD:R_0603_1608Metric"
+		(property "Footprint" "Resistor_SMD:R_0402_1005Metric"
 			(at 302.26 69.342 90)
 			(effects
@@
 			)
 		)
-		(property "Footprint" "Resistor_SMD:R_0603_1608Metric"
+		(property "Footprint" "Resistor_SMD:R_0402_1005Metric"
 			(at 166.878 87.63 90)
 			(effects
@@
 			)
 		)
-		(property "Footprint" "Resistor_SMD:R_0603_1608Metric"
+		(property "Footprint" "Resistor_SMD:R_0402_1005Metric"
 			(at 250.698 87.63 90)
 			(effects
@@
 			)
 		)
-		(property "Footprint" "Resistor_SMD:R_0603_1608Metric"
+		(property "Footprint" "Resistor_SMD:R_0402_1005Metric"
 			(at 218.44 99.822 90)
 			(effects
@@
 			)
 		)
-		(property "Footprint" "Resistor_SMD:R_0603_1608Metric"
+		(property "Footprint" "Resistor_SMD:R_0402_1005Metric"
 			(at 302.26 99.822 90)
 			(effects
@@
 			)
 		)
-		(property "Footprint" "Resistor_SMD:R_0603_1608Metric"
+		(property "Footprint" "Resistor_SMD:R_0402_1005Metric"
 			(at 218.44 59.182 90)
 			(effects
@@
 			)
 		)
-		(property "Footprint" "Resistor_SMD:R_0603_1608Metric"
+		(property "Footprint" "Resistor_SMD:R_0402_1005Metric"
 			(at 260.35 59.182 90)
 			(effects
@@
 			)
 		)
-		(property "Footprint" "Resistor_SMD:R_0603_1608Metric"
+		(property "Footprint" "Resistor_SMD:R_0402_1005Metric"
 			(at 260.35 94.742 90)
 			(effects
@@
 			)
 		)
-		(property "Footprint" "Resistor_SMD:R_0603_1608Metric"
+		(property "Footprint" "Resistor_SMD:R_0402_1005Metric"
 			(at 302.26 94.742 90)
 			(effects
@@
 			)
 		)
-		(property "Footprint" "Resistor_SMD:R_0603_1608Metric"
+		(property "Footprint" "Resistor_SMD:R_0402_1005Metric"
 			(at 302.26 74.422 90)
 			(effects
@@
 			)
 		)
-		(property "Footprint" "Resistor_SMD:R_0603_1608Metric"
+		(property "Footprint" "Resistor_SMD:R_0402_1005Metric"
 			(at 176.53 99.822 90)
 			(effects
@@
 			)
 		)
-		(property "Footprint" "Resistor_SMD:R_0603_1608Metric"
+		(property "Footprint" "Resistor_SMD:R_0402_1005Metric"
 			(at 297.688 87.63 90)
 			(effects
@@
 			)
 		)
-		(property "Footprint" "Resistor_SMD:R_0603_1608Metric"
+		(property "Footprint" "Resistor_SMD:R_0402_1005Metric"
 			(at 171.958 87.63 90)
 			(effects
@@
 			)
 		)
-		(property "Footprint" "Resistor_SMD:R_0603_1608Metric"
+		(property "Footprint" "Resistor_SMD:R_0402_1005Metric"
 			(at 203.708 87.63 90)
 			(effects
@@
 			)
 		)
-		(property "Footprint" "Resistor_SMD:R_0603_1608Metric"
+		(property "Footprint" "Resistor_SMD:R_0402_1005Metric"
 			(at 156.718 87.63 90)
 			(effects
