File: sampling-mesh-monitor/sampling-mesh-monitor.kicad_pcb (KiCad board)
At the start: 6 copper layers, 100 x 100 mm, 264 parts, among them J1 SFP+, J2 USB_C_Receptacle_USB2.0, J3 SWD, Q1 AO3400A, U1 TPS7B4253QPWPRQ1, U10 USBLC6-4SC6, U11 OPA1656, U12 OPA1656, U13 OPA1656, U14 LP2998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

Commit message: Add todos to board schematic
Other:
- copper layers 6 -> 15
