File: sampling-mesh-monitor/sampling-mesh-monitor.kicad_sch (KiCad schematic)
At the start: 276 parts, among them J1 SFP+, J2 USB_C_Receptacle_USB2.0, J3 SWD, Q1 AO3400A, T1 200ps, T10 200ps, T11 200ps, T12 200ps, T2 200ps, T3 200ps, T4 200ps, T5 200ps, T6 200ps, T7 200ps, T8 200ps, T9 200ps, U1 TPS7B4253QPWPRQ1, U10 USBLC6-4SC6, U11 OPA1656, U12 OPA1656, U13 OPA1656, U14 LP2998, U15 AMS1117-3.3, U16 AMS1117-3.3, U17 AMS1117-3.3, U2 74LVC2G157, U3 74LVC2G157, U4 PTN36241B, U5 SKYA21003, U6 SKYA21003, U7 TMUXHS4212, U8 TMUXHS4212, U9 STM32G474RBTx, Y1 8MHz/20p

Commit message: Add todos to board schematic
Other:
- note added: "* Add transistor to LEDs on V_BIAS and V_RES so they work with voltages lower than their 3V V_F * Add cap + 0R tie to AVDD to STM32 VRES+ pin to extend DAC range to AVDD * Hook up 74LVC2G157 such that they can be used either in inv/noninv mode or in AND'ing mode * Switch out driver for PI3HDX12211, add configurable resistors for both pin strapping and I2C options * Remove clip lines? * Clean up a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"
- note added: "TODO:"
