File: uut_meshes_density/uut_meshes.kicad_sch (KiCad schematic)
At the start: 8 parts, among them J1 Conn_02x10_Counter_Clockwise, J2 Conn_02x10_Counter_Clockwise, J3 Conn_02x10_Counter_Clockwise, J4 Conn_02x10_Counter_Clockwise, J5 Conn_02x04_Top_Bottom, J6 Conn_02x04_Top_Bottom, J7 Conn_02x04_Top_Bottom, J8 Conn_02x04_Top_Bottom

Commit message: Add new mesh coupons
Connections:
- net GND: no longer J1.9 (Pin_9), J2.9 (Pin_9), J3.9 (Pin_9), J4.9 (Pin_9)
